File: Nemesis-MixSigPCB.kicad_sch (KiCad schematic)
At the start: 4 parts

Commit message: Add backup file and updates to schematic
Other:
- company: Phil's Lab -> Jacob Parent
- title: Mixed-Signal Demo PCB -> Mixed-Signal PCB
Changed lines of the file:
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@@
 	(paper "A4")
 	(title_block
-		(title "Mixed-Signal Demo PCB")
-		(date "2022-01-04")
+		(title "Mixed-Signal PCB")
+		(date "6-1-2024")
 		(rev "0.1")
-		(company "Phil's Lab")
+		(company "Jacob Parent")
 	)
 	(polyline
