File: ADC.kicad_sch (KiCad schematic)
At the start: 0 parts

Commit message: Adding official files from course download
Parts:
- added C300, C304, C307: 150p, Capacitor_SMD:C_0402_1005Metric, symbol Device:C
- added C301, C302, C306, C311, C313, C314: 100n, Capacitor_SMD:C_0402_1005Metric, symbol Device:C
- added C303, C305: 1n, Capacitor_SMD:C_0402_1005Metric, symbol Device:C
- added C308, C309, C310, C312, C315: 10u, Capacitor_SMD:C_0603_1608Metric, symbol Device:C
- added D300: PESD3V3L1BA,115, Diode_SMD:D_SOD-323, symbol Device:D_TVS
- added J300: 031-5640-1010, PhilsLab_Footprints_KiCad6:AMPHENOL-BNC-031-5640-1010, symbol Connector:Conn_Coaxial
- added R300, R306, R307: 1k, Resistor_SMD:R_0402_1005Metric, symbol Device:R
- added R301, R302: 2M2, Resistor_SMD:R_0402_1005Metric, symbol Device:R
- added R303: 6k8, Resistor_SMD:R_0402_1005Metric, symbol Device:R
- added R304: 22k, Resistor_SMD:R_0402_1005Metric, symbol Device:R
- added R305: 12k, Resistor_SMD:R_0402_1005Metric, symbol Device:R
- added R308: 49R9, Resistor_SMD:R_0402_1005Metric, symbol Device:R
- added R309: 0R, Resistor_SMD:R_0402_1005Metric, symbol Device:R
- added U300, U301: MCP6001T-E/OT, Package_TO_SOT_SMD:SOT-23-5, symbol Amplifier_Operational:MCP6001-OT
- added U302: REF3033AIDBZT, Package_TO_SOT_SMD:SOT-23, symbol Reference_Voltage:REF3033
- added U303: ADC141S626CIMM_NOPB, PhilsLab_Footprints_KiCad6:VSSOP-10, symbol PhilsLab-KiCad-Symbols:ADC141S626CIMM_NOPB
Connections:
- new net: C303.1, R303.1, R304.2
- new net: C305.1, R304.1, R305.2
- new net +3.3VA: C302.1, C306.1, C312.1, C313.1, U300.5 (V+), U301.5 (V+), U303.10 (VA)
- new net +3V3: C314.1, C315.1, U303.9 (VIO)
- new net +5V: C308.1, R308.2
- new net ADC_IN+: C307.1, R306.1, U303.2 (+IN)
- new net ADC_IN-: C307.2, R307.1, U303.3 (-IN)
- new net ADC_SCLK: R309.2, U303.8 (SCLK)
- new net ADC_VREF: C310.1, C311.1, U302.2 (OUT), U303.1 (VREF)
- new net ADC_VREF_VIN: C309.1, R308.1, U302.1 (IN)
- new net GND: C300.2, C302.2, C303.2, C304.2, C306.2, C308.2, C309.2, C310.2, C311.2, C312.2, C313.2, C314.2, C315.2, D300.2 (A2), J300.2 (Ext), R301.1, U300.2 (V-), U301.2 (V-), U302.3 (GND), U303.4 (GND), U303.5 (GND)
- new net IN: D300.1 (A1), J300.1 (In), R300.2
- new net IN_AA_BUF_IN: C304.1, R305.1, U301.3 (+)
- new net IN_AA_BUF_OUT: C305.2, R306.2, U301.1, U301.4 (-)
- new net IN_BUF: C301.1, R302.1, U300.3 (+)
- new net IN_BUF_OUT: R303.2, U300.1, U300.4 (-)
- new net IN_RF: C300.1, C301.2, R300.1, R301.2
- new net SPI1_MISO: U303.7 (DOUT)
- new net SPI1_NSS: U303.6 (NCS)
- new net SPI1_SCK: R309.1
- new net VCOM: R302.2, R307.2
Other:
- note added: "14-Bit S/H ADC"
- note added: "3rd order Butterworth anti-aliasing (low-pass filter) fc=25kHz"
- note added: "Analogue Front-End"
- note added: "BNC connector"
- note added: "Both ADC inputs should be at same VCOM"
- note added: "HP filter: fc=1.4Hz"
- note added: "Input voltage must be in -1.65V to +1.65V range!"
- note added: "MCP6001: I/O Rail-to-Rail, Single-Supply (1V8 to 5V), high-impedance input CMOS, low bias currents, unity gain stable"
- note added: "P(R,max)=0.1W -> I(R,max)=45mA"
- note added: "RF filter: fc=1.1MHz"
- note added: "Rin = 1.1M"
- note added: "Single-ended to 'balanced' conversion"
- note added: "Vref filter: fc=319Hz"
- note added: "Vref=3V3"
- note added: "[3] ADC & Analogue Front-End"
- company: (none) -> Phil's Lab
- title: (none) -> Mixed-Signal Demo PCB

Commit message: Add backup file and updates to schematic
Parts:
- R300, R301, R302, R303, R304, R305, R306, R307, R308, R309: symbol Device:R -> Device:R_US
Other:
- company: Phil's Lab -> Jacob Parent
- title: Mixed-Signal Demo PCB -> Mixed-Signal PCB
Changed lines of the file:
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@@
 	(paper "A4")
 	(title_block
-		(title "Mixed-Signal Demo PCB")
+		(title "Mixed-Signal PCB")
+		(date "6-1-2024")
 		(rev "0.1")
-		(company "Phil's Lab")
+		(company "Jacob Parent")
 	)
 	(junction
@@
 	)
 	(symbol
-		(lib_id "Device:R")
+		(lib_id "Device:R_US")
 		(at 158.75 140.97 270)
 		(unit 1)
@@
 		)
 		(property "Footprint" "Resistor_SMD:R_0402_1005Metric"
-			(at 158.75 139.192 90)
+			(at 158.496 141.986 90)
 			(effects
 				(font
@@
 			)
 		)
-		(property "Description" ""
+		(property "Description" "Resistor, US symbol"
 			(at 158.75 140.97 0)
 			(effects
@@
 	)
 	(symbol
-		(lib_id "Device:R")
+		(lib_id "Device:R_US")
 		(at 64.77 62.23 270)
 		(unit 1)
@@
 		)
 		(property "Footprint" "Resistor_SMD:R_0402_1005Metric"
-			(at 64.77 60.452 90)
+			(at 64.516 63.246 90)
 			(effects
 				(font
@@
 			)
 		)
-		(property "Description" ""
+		(property "Description" "Resistor, US symbol"
 			(at 64.77 62.23 0)
 			(effects
@@
 	)
 	(symbol
-		(lib_id "Device:R")
+		(lib_id "Device:R_US")
 		(at 71.12 68.58 180)
 		(unit 1)
@@
 		)
 		(property "Footprint" "Resistor_SMD:R_0402_1005Metric"
-			(at 72.898 68.58 90)
+			(at 70.104 68.326 90)
 			(effects
 				(font
@@
 			)
 		)
-		(property "Description" ""
+		(property "Description" "Resistor, US symbol"
 			(at 71.12 68.58 0)
 			(effects
@@
 	)
 	(symbol
-		(lib_id "Device:R")
+		(lib_id "Device:R_US")
 		(at 100.33 55.88 180)
 		(unit 1)
@@
 		)
 		(property "Footprint" "Resistor_SMD:R_0402_1005Metric"
-			(at 102.108 55.88 90)
+			(at 99.314 55.626 90)
 			(effects
 				(font
@@
 			)
 		)
-		(property "Description" ""
+		(property "Description" "Resistor, US symbol"
 			(at 100.33 55.88 0)
 			(effects
@@
 	)
 	(symbol
-		(lib_id "Device:R")
+		(lib_id "Device:R_US")
 		(at 153.67 64.77 270)
 		(unit 1)
@@
 		)
 		(property "Footprint" "Resistor_SMD:R_0402_1005Metric"
-			(at 153.67 62.992 90)
+			(at 153.416 65.786 90)
 			(effects
 				(font
@@
 			)
 		)
-		(property "Description" ""
+		(property "Description" "Resistor, US symbol"
 			(at 153.67 64.77 0)
 			(effects
@@
 	)
 	(symbol
-		(lib_id "Device:R")
+		(lib_id "Device:R_US")
 		(at 166.37 64.77 270)
 		(unit 1)
@@
 		)
 		(property "Footprint" "Resistor_SMD:R_0402_1005Metric"
-			(at 166.37 62.992 90)
+			(at 166.116 65.786 90)
 			(effects
 				(font
@@
 			)
 		)
-		(property "Description" ""
+		(property "Description" "Resistor, US symbol"
 			(at 166.37 64.77 0)
 			(effects
@@
 	)
 	(symbol
-		(lib_id "Device:R")
+		(lib_id "Device:R_US")
 		(at 179.07 64.77 270)
 		(unit 1)
@@
 		)
 		(property "Footprint" "Resistor_SMD:R_0402_1005Metric"
-			(at 179.07 62.992 90)
+			(at 178.816 65.786 90)
 			(effects
 				(font
@@
 			)
 		)
-		(property "Description" ""
+		(property "Description" "Resistor, US symbol"
 			(at 179.07 64.77 0)
 			(effects
@@
 	)
 	(symbol
-		(lib_id "Device:R")
+		(lib_id "Device:R_US")
 		(at 236.22 67.31 270)
 		(unit 1)
@@
 		)
 		(property "Footprint" "Resistor_SMD:R_0402_1005Metric"
-			(at 236.22 65.532 90)
+			(at 235.966 68.326 90)
 			(effects
 				(font
@@
 			)
 		)
-		(property "Description" ""
+		(property "Description" "Resistor, US symbol"
 			(at 236.22 67.31 0)
 			(effects
@@
 	)
 	(symbol
-		(lib_id "Device:R")
+		(lib_id "Device:R_US")
 		(at 236.22 87.63 270)
 		(unit 1)
@@
 		)
 		(property "Footprint" "Resistor_SMD:R_0402_1005Metric"
-			(at 236.22 85.852 90)
+			(at 235.966 88.646 90)
 			(effects
 				(font
@@
 			)
 		)
-		(property "Description" ""
+		(property "Description" "Resistor, US symbol"
 			(at 236.22 87.63 0)
 			(effects
@@
 	)
 	(symbol
-		(lib_id "Device:R")
+		(lib_id "Device:R_US")
 		(at 49.53 135.89 270)
 		(unit 1)
@@
 		)
 		(property "Footprint" "Resistor_SMD:R_0402_1005Metric"
-			(at 49.53 134.112 90)
+			(at 49.276 136.906 90)
 			(effects
 				(font
@@
 			)
 		)
-		(property "Description" ""
+		(property "Description" "Resistor, US symbol"
 			(at 49.53 135.89 0)
 			(effects

Commit message: Add files via upload
Parts:
- J300: footprint PhilsLab_Footprints_KiCad6:AMPHENOL-BNC-031-5640-1010 -> MixedSignalBoardParts:BNC
- U303: footprint PhilsLab_Footprints_KiCad6:VSSOP-10 -> MixedSignalBoardParts:SOIC-10
Changed lines of the file:
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@@
 			)
 		)
-		(property "Footprint" "PhilsLab_Footprints_KiCad6:VSSOP-10"
+		(property "Footprint" "MixedSignalBoardParts:SOIC-10"
 			(at 130.81 156.21 0)
 			(effects
@@
 			)
 		)
-		(property "Footprint" "PhilsLab_Footprints_KiCad6:AMPHENOL-BNC-031-5640-1010"
+		(property "Footprint" "MixedSignalBoardParts:BNC"
 			(at 45.72 62.23 0)
 			(effects
@@
 			)
 		)
-		(property "Datasheet" " ~"
+		(property "Datasheet" "~"
 			(at 45.72 62.23 0)
 			(effects
