File: Nemesis-MixSigPCB.kicad_pcb (KiCad board)
At the start: 2 copper layers, 114 parts, among them J200 USB_C_Receptacle_USB2.0, J201 2x5 1.27mm, J300 031-5640-1010, J400 031-5640-1010, U100 HT7533-1, U101 TLV62569DBV, U102 MCP6001T-E/OT, U200 STM32F103CBT6, U201 USBLC6-2SC6, U300 MCP6001T-E/OT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

Commit message: Layout Complete
Still need to add assembly files
Parts:
- added G***: LOGO, LOGO, F.Cu at (188.5, 105.8)
- moved H3 183.4 mm to (192.5, 124.8)
- moved H4 164.7 mm to (192.5, 59.8)
- moved R205 152.8 mm to (193.8, 86.2), turned to 180 degrees
- moved J200 152.6 mm to (195.2, 79.7), turned to 90 degrees
- moved R206 148.7 mm to (193.9, 73.2), turned to 180 degrees
- moved U201 146.7 mm to (185.5, 79.2), turned to 180 degrees
- moved H2 145.1 mm to (142.5, 124.8)
- moved J201 141.9 mm to (157.7, 60.3), turned to -90 degrees
- moved U200 137.6 mm to (167.5, 80.2)
- moved R405 136.8 mm to (180.2, 110.2), turned to 90 degrees
- moved C404 136.7 mm to (180.7, 107.7)
- moved R401 134.8 mm to (178.8, 100.7)
- moved R404 134.6 mm to (179.0, 106.1), turned to 180 degrees
- moved R403 134.2 mm to (177.5, 105.6), turned to 90 degrees
- moved R202 133.7 mm to (173.6, 83.8), turned to 90 degrees
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Connections:
- J300 pad 3: (no net) -> GND
- J300 pad 4: (no net) -> GND
- J400 pad 3: (no net) -> GND
- J400 pad 4: (no net) -> GND
Routing:
- net +3V3: track 0.00 -> 174.3 mm, vias 0 -> 15
- net +5V: track 0.00 -> 76.6 mm, vias 0 -> 4
- net +3.3VA: track 0.00 -> 63.6 mm, vias 0 -> 3
- net GND: track 0.00 -> 52.9 mm, vias 0 -> 396
- net /MCU/TIM4_CH1: track 0.00 -> 31.3 mm, vias 0 -> 2
- net /MCU/TIM4_CH2: track 0.00 -> 28.1 mm, vias 0 -> 2
- net /MCU/NRST: track 0.00 -> 26.6 mm, vias 0 -> 2
- net /MCU/TIM4_CH3: track 0.00 -> 26.2 mm, vias 0 -> 2
- net SPI2_MOSI: track 0.00 -> 26.0 mm
- net DAC_NCLR: track 0.00 -> 25.6 mm, vias 0 -> 2
- net DAC_NLDAC: track 0.00 -> 25.3 mm, vias 0 -> 2
- net VCOM: track 0.00 -> 24.1 mm
- net /MCU/SWDIO: track 0.00 -> 22.5 mm
- net VBUS: track 0.00 -> 22.1 mm
- net SPI1_MISO: track 0.00 -> 21.7 mm
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- added copper zone on F.Cu, net +3.3VA
- added copper zone on F.Cu, net +3V3
- added copper zone on F.Cu, net +5V
- added copper zone on F.Cu, net /ADC/ADC_VREF
- added copper zone on F.Cu, net /ADC/ADC_VREF_VIN
- added copper zone on F.Cu, net /Power/+5V_FILT
- added copper zone on F.Cu, net /Power/BUCK_SW
- added copper zone on F.Cu, net GND
- added copper zone on In1.Cu, net GND
- added copper zone on F.Cu, net VBUS
- added copper zone on F.Cu, net VDDA
Other:
- board outline added: 60 x 75 mm
- copper layers 2 -> 4
- board text added: "1 MOhm"
- board text added: "20 -> 20kHz"
- board text added: "50 Ohm"
- board text added: "IN"
- board text added: "JCP 8/18/24 REV A"
- board text added: "Mixed Signal Demo Board"
- board text added: "ON"
- board text added: "OUT"
- board text added: "S"
- board text added: "SWD"
- board text added: "USB"
- board text added: "www.jacobcparent.com"
